File: Mainboard/macropad.kicad_pcb (KiCad board)
At the start: 2 copper layers, 48.3 x 40.6 mm, 45 parts, among them J1 SWD, J11 Keyboard 1, J12 Keyboard 2, J13 Keyboard 2, J4 Keyboard 1, J5 UART, J6 RS485, J7 Extra, J8 USB_A, J9 CAN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

Commit message: Cleaned up project structure.
Other:
- board text added: "GND CANL CANH 5V"
- board text removed: "5V CANH CANL GND"
Changed lines of the file:
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@@
 		)
 	)
-	(gr_text "\n5V\nCANH\nCANL\nGND"
+	(gr_text "GND\nCANL\nCANH\n5V\n"
 		(at 96.313289 94.848065 0)
 		(layer "B.SilkS")
@@
 	)
 	(gr_text "*CAN*"
-		(at 99.605 87.545 0)
+		(at 100.170588 87.78183 0)
 		(layer "B.SilkS")
 		(effects
